Commit message: feat: prep canonical phoxal-cli test bed
- identity.id: sandbox-rover → robot-rover (matches repo name; sets docker
  compose project name now that phoxal-cli writes name: <robot_id>)
- cli_min_version: ^0.6 → >=0.0.0-0 (admit dev + future versions)
- phoxal_runtimes.version: ^0.1 → latest (track newest framework release)
- structure.urdf: add four <name>_drive__motor_joint continuous joints with
  matching cylinder wheel links (r=0.1 m matches wheel_radius_m). Required
  for the ddsm115 encoder targets to resolve.
- sim/worlds/default.wbt: seeded from framework's ArenaWorld.wbt fixture
- phoxal.lock: pinned to framework v0.2.0 multi-arch index digests +
  simulator v0.2.0 + operator/joypad v0.1.0

Verified end-to-end: phoxal-cli v0.1.2 doctor --fix downloads all four
cached tools, simulate --dry-run --locked stages the .phoxal/run and
.phoxal/webots trees, and docker compose -f .phoxal/run/docker-compose.yml
up -d brings up all 18 platform-runtime services healthy (named
robot-rover-<service>-1, including odometry).

Signed-off-by: jbernavaprah <webjure@gmail.com>

File: structure.urdf (robot description, URDF)
Before this commit: robot RgbdImuDiffDrive, 10 links, 9 joints
Links:
- added link front_left_wheel, mass 0.5; collision cylinder length=0.05 radius=0.1; visual cylinder length=0.05 radius=0.1
- added link front_right_wheel, mass 0.5; collision cylinder length=0.05 radius=0.1; visual cylinder length=0.05 radius=0.1
- added link rear_left_wheel, mass 0.5; collision cylinder length=0.05 radius=0.1; visual cylinder length=0.05 radius=0.1
- added link rear_right_wheel, mass 0.5; collision cylinder length=0.05 radius=0.1; visual cylinder length=0.05 radius=0.1
Joints:
- added joint front_left_drive__motor_joint: type continuous, parent front_left_wheel_mount, child front_left_wheel, origin xyz=0 0 0 rpy=0 0 0, axis 0 0 1
- added joint front_right_drive__motor_joint: type continuous, parent front_right_wheel_mount, child front_right_wheel, origin xyz=0 0 0 rpy=0 0 0, axis 0 0 1
- added joint rear_left_drive__motor_joint: type continuous, parent rear_left_wheel_mount, child rear_left_wheel, origin xyz=0 0 0 rpy=0 0 0, axis 0 0 1
- added joint rear_right_drive__motor_joint: type continuous, parent rear_right_wheel_mount, child rear_right_wheel, origin xyz=0 0 0 rpy=0 0 0, axis 0 0 1
