Commit message: chore: adopt framework train 0.45.2
Framework 0.45.1 (#362) reserves '__' as the component-instance
namespacing separator and composes each component's own structure at its
mount link. Drop the hand-authored wheel links and '<instance>__motor_joint'
joints from the robot URDF: the ddsm115 component structure now supplies
the wheel (mount -> motor_joint -> rotor_link) at every '*_wheel_mount'.

Verified: cargo check green and 'phoxal validate' (which runs the same
resolve+compile step that 'run' failed in) passes on phoxal 0.29.4.

File: structure.urdf (robot description, URDF)
Before this commit: robot RgbdImuDiffDrive, 14 links, 13 joints
Links:
- removed link front_left_wheel
- removed link front_right_wheel
- removed link rear_left_wheel
- removed link rear_right_wheel
Joints:
- removed joint front_left_drive__motor_joint
- removed joint front_right_drive__motor_joint
- removed joint rear_left_drive__motor_joint
- removed joint rear_right_drive__motor_joint
